File: pcb/polar_sketcher.kicad_pcb (KiCad board)
At the start: 2 copper layers, 125.2 x 66.2 mm, 31 parts, among them J1 LIMIT_1, J10 SERVO_PINS, J11 ENCODER, J12 ESP_H_1, J13 RPi_H_1, J14 RPi_H_2, J2 LIMIT_3, J3 STEPPER_1, J4 ESP_H_1, J5 ESP_H_2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

Commit message: fix design flaw in PCB that makes it fry the esp32 if you connect the encoder the opposite way around
Parts:
- removed RaspberryPi Spares: RPi_H_1, Connector_PinSocket_2.54mm:PinSocket_1x14_P2.54mm_Vertical
- added RaspberryPiSpares1: RPi_H_1, Connector_PinSocket_2.54mm:PinSocket_1x14_P2.54mm_Vertical, F.Cu at (217.3, 111.5)
- ESP32Power1: value 3.3V -> V+
Connections:
- J11 pad 5: GND -> GND2
Routing:
- net GND2: track 76.5 -> 102.0 mm
- net GND: track 99.2 -> 96.7 mm, vias 18 -> 17
